File: DMH_BBDelay_PANEL/DMH_BBDelay_PANEL.kicad_sch (KiCad schematic)
At the start: 34 parts, among them J0 Panel_GND_Solder_Wire_Pad

Commit message: FInalized panel design
Parts:
- H18: value Clock Sync A -> Clk Sync A
- H19: value Clock Sync B -> Clk Sync B
- H20: value Input A -> In A
- H21: value Input B -> In B
- H22: value Output A -> Out A
- H23: value Output B -> Out B
- H25: value FB CV B -> FB B CV
- H34: value Clock A -> Clk A
- H35: value Clock B -> Clk B
- H5: value Time A&B -> Time
- H7: value FB CV A -> FB A CV
Changed lines of the file:
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@@
 			)
 		)
-		(property "Value" "FB CV A"
+		(property "Value" "FB A CV"
 			(at 78.74 38.1 0)
 			(effects
@@
 			)
 		)
-		(property "Value" "Time A&B"
+		(property "Value" "Time"
 			(at 53.34 25.4 0)
 			(effects
@@
 			)
 		)
-		(property "Value" "Input A"
+		(property "Value" "In A"
 			(at 27.94 114.3 0)
 			(effects
@@
 			)
 		)
-		(property "Value" "Input B"
+		(property "Value" "In B"
 			(at 27.94 127 0)
 			(effects
@@
 			)
 		)
-		(property "Value" "Output B"
+		(property "Value" "Out B"
 			(at 53.34 127 0)
 			(effects
@@
 			)
 		)
-		(property "Value" "FB CV B"
+		(property "Value" "FB B CV"
 			(at 104.14 38.1 0)
 			(effects
@@
 			)
 		)
-		(property "Value" "Clock Sync B"
+		(property "Value" "Clk Sync B"
 			(at 104.14 88.9 0)
 			(effects
@@
 			)
 		)
-		(property "Value" "Output A"
+		(property "Value" "Out A"
 			(at 53.34 114.3 0)
 			(effects
@@
 			)
 		)
-		(property "Value" "Clock Sync A"
+		(property "Value" "Clk Sync A"
 			(at 104.14 76.2 0)
 			(effects
@@
 			)
 		)
-		(property "Value" "Clock B"
+		(property "Value" "Clk B"
 			(at 180.34 127 0)
 			(effects
@@
 			)
 		)
-		(property "Value" "Clock A"
+		(property "Value" "Clk A"
 			(at 180.34 114.3 0)
 			(effects

Commit message: Added LEDs and Link switch
Parts:
- added H28: LED_A, SynthStuff:MountingHole_LED_3mm_R, symbol Mechanical:MountingHole
- added H29: LED_B, SynthStuff:MountingHole_LED_3mm_R, symbol Mechanical:MountingHole
- added H36: Link, SynthStuff:Toggle_Switch_TE_Cutout, symbol SynthStuff:MountingHole_ToggleSwitch
- H12: value Input Gain A -> A
- H13: value Input Gain B -> B
Connections:
- net GND: now also H36.1
Changed lines of the file:
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@@
+	)
+	(junction
+		(at 101.6 57.15)
+		(diameter 0)
+		(color 0 0 0 0)
 	)
 	(junction
@@
 	(wire
 		(pts
+			(xy 152.4 54.61) (xy 152.4 57.15)
+		)
+		(stroke
+			(width 0)
+			(type default)
+		)
+	)
+	(wire
+		(pts
 			(xy 120.65 101.6) (xy 120.65 114.3)
 		)
@@
 		(pts
 			(xy 69.85 114.3) (xy 72.39 114.3)
+		)
+		(stroke
+			(width 0)
+			(type default)
+		)
+	)
+	(wire
+		(pts
+			(xy 152.4 57.15) (xy 101.6 57.15)
 		)
 		(stroke
@@
 			)
 		)
-		(property "Value" "Input Gain A"
+		(property "Value" "A"
 			(at 104.14 50.8 0)
 			(effects
@@
 	)
 	(symbol
+		(lib_id "SynthStuff:MountingHole_ToggleSwitch")
+		(at 152.4 50.8 0)
+		(unit 1)
+		(exclude_from_sim yes)
+		(in_bom no)
+		(on_board yes)
+		(dnp no)
+		(fields_autoplaced yes)
+		(property "Reference" "H36"
+			(at 154.94 48.2599 0)
+			(effects
+				(font
+					(size 1.27 1.27)
+				)
+				(justify left)
+			)
+		)
+		(property "Value" "Link"
+			(at 154.94 50.8 0)
+			(effects
+				(font
+					(size 1.27 1.27)
+					(thickness 0.254)
+					(bold yes)
+					(italic yes)
+				)
+				(justify left)
+			)
+		)
+		(property "Footprint" "SynthStuff:Toggle_Switch_TE_Cutout"
+			(at 152.4 50.8 0)
+			(effects
+				(font
+					(size 1.27 1.27)
+				)
+				(hide yes)
+			)
+		)
+		(property "Datasheet" "~"
+			(at 152.4 50.8 0)
+			(effects
+				(font
+					(size 1.27 1.27)
+				)
+				(hide yes)
+			)
+		)
+		(property "Description" "Toggle Switch Mounting Hole"
+			(at 154.94 53.3399 0)
+			(effects
+				(font
+					(size 1.27 1.27)
+				)
+				(justify left)
+			)
+		)
+		(property "Function" ""
+			(at 152.4 50.8 0)
+			(effects
+				(font
+					(size 1.27 1.27)
+				)
+			)
+		)
+		(pin "1"
+		)
+		(instances
+			(project "DMH_BBDelay_PANEL"
+				(path "/a552705f-a9fe-462e-9913-5cfcc08b233c"
+					(reference "H36")
+					(unit 1)
+				)
+			)
+		)
+	)
+	(symbol
 		(lib_id "SynthStuff:MountingHole_Jack6.35mm_v2")
 		(at 76.2 114.3 0)
@@
 				(path "/a552705f-a9fe-462e-9913-5cfcc08b233c"
 					(reference "H26")
+					(unit 1)
+				)
+			)
+		)
+	)
+	(symbol
+		(lib_id "Mechanical:MountingHole")
+		(at 177.8 38.1 0)
+		(unit 1)
+		(exclude_from_sim no)
+		(in_bom no)
+		(on_board yes)
+		(dnp no)
+		(fields_autoplaced yes)
+		(property "Reference" "H29"
+			(at 180.34 36.8299 0)
+			(effects
+				(font
+					(size 1.27 1.27)
+				)
+				(justify left)
+			)
+		)
+		(property "Value" "LED_B"
+			(at 180.34 39.37 0)
+			(effects
+				(font
+					(size 1.27 1.27)
+					(thickness 0.254)
+					(bold yes)
+					(italic yes)
+				)
+				(justify left)
+			)
+		)
+		(property "Footprint" "SynthStuff:MountingHole_LED_3mm_R"
+			(at 177.8 38.1 0)
+			(effects
+				(font
+					(size 1.27 1.27)
+				)
+				(hide yes)
+			)
+		)
+		(property "Datasheet" "~"
+			(at 177.8 38.1 0)
+			(effects
+				(font
+					(size 1.27 1.27)
+				)
+				(hide yes)
+			)
+		)
+		(property "Description" "Mounting Hole without connection"
+			(at 177.8 38.1 0)
+			(effects
+				(font
+					(size 1.27 1.27)
+				)
+				(hide yes)
+			)
+		)
+		(instances
+			(project ""
+				(path "/a552705f-a9fe-462e-9913-5cfcc08b233c"
+					(reference "H29")
 					(unit 1)
 				)
@@
 			)
 		)
-		(property "Value" "Input Gain B"
+		(property "Value" "B"
 			(at 104.14 63.5 0)
 			(effects
@@
 					(unit 1)
 				)
+			)
+		)
+	)
+	(symbol
+		(lib_id "Mechanical:MountingHole")
+		(at 152.4 38.1 0)
+		(unit 1)
+		(exclude_from_sim no)
+		(in_bom no)
+		(on_board yes)
+		(dnp no)
+		(fields_autoplaced yes)
+		(property "Reference" "H28"
+			(at 154.94 36.8299 0)
+			(effects
+				(font
+					(size 1.27 1.27)
+				)
+				(justify left)
+			)
+		)
+		(property "Value" "LED_A"
+			(at 154.94 39.37 0)
+			(effects
+				(font
+					(size 1.27 1.27)
+					(thickness 0.254)
+					(bold yes)
+					(italic yes)
+				)
+				(justify left)
+			)
+		)
+		(property "Footprint" "SynthStuff:MountingHole_LED_3mm_R"
+			(at 152.4 38.1 0)
+			(effects
+				(font
+					(size 1.27 1.27)
+				)
+				(hide yes)
+			)
+		)
+		(property "Datasheet" "~"
+			(at 152.4 38.1 0)
+			(effects
+				(font
+					(size 1.27 1.27)
+				)
+				(hide yes)
+			)
+		)
+		(property "Description" "Mounting Hole without connection"
+			(at 152.4 38.1 0)
+			(effects
+				(font
+					(size 1.27 1.27)
+				)
+				(hide yes)
+			)
+		)
+		(instances
+			(project ""
+				(path "/a552705f-a9fe-462e-9913-5cfcc08b233c"
+					(reference "H28")
+					(unit 1)
+				)

Commit message: Added tone knob
... by making Input Gain switch to span both channels. Also added a center Linked LED
Parts:
- added H37: Tone, SynthStuff:Pot_Cutout_Tiny_text_P110KH1, symbol SynthStuff:MountingHole_Pot
- added H38: LED_L, SynthStuff:MountingHole_LED_3mm_B, symbol Mechanical:MountingHole
- H12: value A -> Gain
- H13: now not fitted
Connections:
- net GND: now also H37.1
Other:
- moved on the sheet: H28, H29
Changed lines of the file:
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@@
+	)
+	(junction
+		(at 101.6 69.85)
+		(diameter 0)
+		(color 0 0 0 0)
 	)
 	(junction
@@
 	(wire
 		(pts
+			(xy 152.4 67.31) (xy 152.4 69.85)
+		)
+		(stroke
+			(width 0)
+			(type default)
+		)
+	)
+	(wire
+		(pts
 			(xy 19.05 259.08) (xy 27.94 259.08)
 		)
@@
 		(pts
 			(xy 76.2 92.71) (xy 76.2 101.6)
+		)
+		(stroke
+			(width 0)
+			(type default)
+		)
+	)
+	(wire
+		(pts
+			(xy 101.6 69.85) (xy 152.4 69.85)
 		)
 		(stroke
@@
 			)
 		)
-		(property "Value" "A"
+		(property "Value" "Gain"
 			(at 104.14 50.8 0)
 			(effects
@@
 	)
 	(symbol
+		(lib_id "SynthStuff:MountingHole_Pot")
+		(at 152.4 64.77 0)
+		(unit 1)
+		(exclude_from_sim yes)
+		(in_bom yes)
+		(on_board yes)
+		(dnp no)
+		(fields_autoplaced yes)
+		(property "Reference" "H37"
+			(at 154.94 60.9599 0)
+			(effects
+				(font
+					(size 1.27 1.27)
+				)
+				(justify left)
+			)
+		)
+		(property "Value" "Tone"
+			(at 154.94 63.5 0)
+			(effects
+				(font
+					(size 1.27 1.27)
+					(thickness 0.254)
+					(bold yes)
+					(italic yes)
+				)
+				(justify left)
+			)
+		)
+		(property "Footprint" "SynthStuff:Pot_Cutout_Tiny_text_P110KH1"
+			(at 152.4 64.77 0)
+			(effects
+				(font
+					(size 1.27 1.27)
+				)
+				(hide yes)
+			)
+		)
+		(property "Datasheet" "~"
+			(at 152.4 64.77 0)
+			(effects
+				(font
+					(size 1.27 1.27)
+				)
+				(hide yes)
+			)
+		)
+		(property "Description" "Pot Mounting Hole"
+			(at 154.94 66.0399 0)
+			(effects
+				(font
+					(size 1.27 1.27)
+				)
+				(justify left)
+			)
+		)
+		(pin "1"
+		)
+		(instances
+			(project "DMH_BBDelay_PANEL"
+				(path "/a552705f-a9fe-462e-9913-5cfcc08b233c"
+					(reference "H37")
+					(unit 1)
+				)
+			)
+		)
+	)
+	(symbol
 		(lib_id "SynthStuff:MountingHole_ToggleSwitch")
 		(at 152.4 50.8 0)
@@
 	(symbol
 		(lib_id "Mechanical:MountingHole")
-		(at 177.8 38.1 0)
+		(at 177.8 25.4 0)
 		(unit 1)
 		(exclude_from_sim no)
@@
 		(fields_autoplaced yes)
 		(property "Reference" "H29"
-			(at 180.34 36.8299 0)
+			(at 180.34 24.1299 0)
 			(effects
 				(font
@@
 		)
 		(property "Value" "LED_B"
-			(at 180.34 39.37 0)
+			(at 180.34 26.67 0)
 			(effects
 				(font
@@
 		)
 		(property "Footprint" "SynthStuff:MountingHole_LED_3mm_R"
-			(at 177.8 38.1 0)
+			(at 177.8 25.4 0)
 			(effects
 				(font
@@
 		)
 		(property "Datasheet" "~"
-			(at 177.8 38.1 0)
+			(at 177.8 25.4 0)
 			(effects
 				(font
@@
 		)
 		(property "Description" "Mounting Hole without connection"
-			(at 177.8 38.1 0)
+			(at 177.8 25.4 0)
 			(effects
 				(font
@@
 		(exclude_from_sim yes)
 		(in_bom no)
-		(on_board yes)
-		(dnp no)
+		(on_board no)
+		(dnp yes)
 		(fields_autoplaced yes)
 		(property "Reference" "H13"
@@
 	(symbol
 		(lib_id "Mechanical:MountingHole")
-		(at 152.4 38.1 0)
+		(at 165.1 38.1 0)
+		(unit 1)
+		(exclude_from_sim no)
+		(in_bom no)
+		(on_board yes)
+		(dnp no)
+		(fields_autoplaced yes)
+		(property "Reference" "H38"
+			(at 167.64 36.8299 0)
+			(effects
+				(font
+					(size 1.27 1.27)
+				)
+				(justify left)
+			)
+		)
+		(property "Value" "LED_L"
+			(at 167.64 39.37 0)
+			(effects
+				(font
+					(size 1.27 1.27)
+					(thickness 0.254)
+					(bold yes)
+					(italic yes)
+				)
+				(justify left)
+			)
+		)
+		(property "Footprint" "SynthStuff:MountingHole_LED_3mm_B"
+			(at 165.1 38.1 0)
+			(effects
+				(font
+					(size 1.27 1.27)
+				)
+				(hide yes)
+			)
+		)
+		(property "Datasheet" "~"
+			(at 165.1 38.1 0)
+			(effects
+				(font
+					(size 1.27 1.27)
+				)
+				(hide yes)
+			)
+		)
+		(property "Description" "Mounting Hole without connection"
+			(at 165.1 38.1 0)
+			(effects
+				(font
+					(size 1.27 1.27)
+				)
+				(hide yes)
+			)
+		)
+		(property "Function" ""
+			(at 165.1 38.1 0)
+			(effects
+				(font
+					(size 1.27 1.27)
+				)
+			)
+		)
+		(instances
+			(project "DMH_BBDelay_PANEL"
+				(path "/a552705f-a9fe-462e-9913-5cfcc08b233c"
+					(reference "H38")
+					(unit 1)
+				)
+			)
+		)
+	)
+	(symbol
+		(lib_id "Mechanical:MountingHole")
+		(at 152.4 25.4 0)
 		(unit 1)
 		(exclude_from_sim no)
@@
 		(fields_autoplaced yes)
 		(property "Reference" "H28"
-			(at 154.94 36.8299 0)
+			(at 154.94 24.1299 0)
 			(effects
 				(font
@@
 		)
 		(property "Value" "LED_A"
-			(at 154.94 39.37 0)
+			(at 154.94 26.67 0)
 			(effects
 				(font
@@
 		)
 		(property "Footprint" "SynthStuff:MountingHole_LED_3mm_R"
-			(at 152.4 38.1 0)
+			(at 152.4 25.4 0)
 			(effects
 				(font
@@
 		)
 		(property "Datasheet" "~"
-			(at 152.4 38.1 0)
+			(at 152.4 25.4 0)
 			(effects
 				(font
@@
 		)
 		(property "Description" "Mounting Hole without connection"
-			(at 152.4 38.1 0)
-			(effects
-				(font
+			(at 152.4 25.4 0)
+			(effects
+				(font
