File: DMH_BBDelay_PANEL/DMH_BBDelay_PANEL.kicad_pcb (KiCad board)
At the start: 2 copper layers, 100 x 200 mm, 38 parts, among them J0 Panel_GND_Solder_Wire_Pad

Commit message: Schematic in progress
Parts:
- H12: value Gain -> PP
Changed lines of the file:
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@@
 			)
 		)
-		(property "Value" "Gain"
+		(property "Value" "PP"
 			(at 0 9.2 0)
 			(unlocked yes)
@@
 				)
 			)
-			(render_cache "Gain" 0
+			(render_cache "PP" 0
 				(polygon
 					(pts
-						(xy 87.868127 101.53) (xy 87.908424 101.526073) (xy 87.940421 101.514219) (xy 87.96099 101.498023)
-						(xy 87.975817 101.476068) (xy 87.988538 101.40971) (xy 87.988538 100.494898) (xy 87.484543 100.494898)
-						(xy 87.484543 101.000969) (xy 87.480529 101.023902) (xy 87.468063 101.03647) (xy 87.448151 101.040048)
-						(xy 86.963695 101.040048) (xy 86.890677 101.036253) (xy 86.824467 101.025317) (xy 86.764441 101.007812)
-						(xy 86.710607 100.984461) (xy 86.617156 100.920318) (xy 86.582921 100.886297) (xy 86.546146 100.841015)
-						(xy 86.515506 100.790905) (xy 86.491697 100.736916) (xy 86.475166 100.679528) (xy 86.465318 100.5871)
-						(xy 86.480344 100.47238) (xy 86.524845 100.364483) (xy 86.557481 100.31557) (xy 86.596173 100.271628)
-						(xy 86.605269 100.262868) (xy 86.653477 100.223763) (xy 86.708433 100.191226) (xy 86.763206 100.168752)
-						(xy 86.825317 100.152381) (xy 86.963695 100.139891) (xy 87.98573 100.139891) (xy 87.98573 99.638583)
-						(xy 86.963695 99.638583) (xy 86.859816 99.642432) (xy 86.76218 99.653747) (xy 86.671475 99.671962)
-						(xy 86.586524 99.696811) (xy 86.506857 99.728084) (xy 86.432617 99.765355) (xy 86.297086 99.858664)
-						(xy 86.263695 99.887833) (xy 86.148157 100.016028) (xy 86.099432 100.087572) (xy 86.057242 100.163542)
-						(xy 86.022354 100.242582) (xy 85.994645 100.325114) (xy 85.974824 100.409045) (xy 85.962656 100.495546)
-						(xy 85.958514 100.584291) (xy 85.973694 100.756851) (xy 86.018549 100.921229) (xy 86.091713 101.073641)
-						(xy 86.191025 101.209638) (xy 86.202146 101.222009) (xy 86.262923 101.282846) (xy 86.329442 101.337887)
-						(xy 86.398964 101.385027) (xy 86.474008 101.426135) (xy 86.552787 101.46017) (xy 86.637033 101.487823)
-						(xy 86.726122 101.508653) (xy 86.820779 101.522602) (xy 86.963695 101.53)
+						(xy 89.319913 99.649453) (xy 89.401579 99.664902) (xy 89.47595 99.686626) (xy 89.545429 99.715156)
+						(xy 89.608359 99.74957) (xy 89.670123 99.793281) (xy 89.725594 99.843014) (xy 89.800426 99.931132)
+						(xy 89.874844 100.061146) (xy 89.920322 100.201712) (xy 89.93552 100.346032) (xy 89.934469 100.383887)
+						(xy 89.926224 100.458421) (xy 89.91013 100.531076) (xy 89.885975 100.602888) (xy 89.854469 100.67162)
+						(xy 89.815729 100.737193) (xy 89.770412 100.798492) (xy 89.731809 100.841013) (xy 89.623256 100.930127)
+						(xy 89.561851 100.965895) (xy 89.494497 100.996097) (xy 89.421004 101.020306) (xy 89.34101 101.038165)
+						(xy 89.252719 101.049399) (xy 89.157118 101.053237) (xy 88.286393 101.053237) (xy 88.286393 101.53)
+						(xy 87.779589 101.53) (xy 87.779589 100.178848) (xy 88.286393 100.178848) (xy 88.286393 100.588443)
+						(xy 89.168353 100.588443) (xy 89.237978 100.583348) (xy 89.283935 100.572341) (xy 89.322494 100.555599)
+						(xy 89.358026 100.530522) (xy 89.386707 100.499295) (xy 89.416827 100.446432) (xy 89.427734 100.40797)
+						(xy 89.431525 100.365572) (xy 89.422282 100.297764) (xy 89.406669 100.258598) (xy 89.383898 100.223422)
+						(xy 89.351887 100.192248) (xy 89.318495 100.170819) (xy 89.278246 100.154504) (xy 89.228027 100.143672)
+						(xy 89.168353 100.139891) (xy 88.322785 100.139891) (xy 88.300794 100.145245) (xy 88.290147 100.157832)
+						(xy 88.286393 100.178848) (xy 87.779589 100.178848) (xy 87.779589 99.756186) (xy 87.792716 99.692338)
+						(xy 87.808276 99.670423) (xy 87.829754 99.654214) (xy 87.862322 99.642491) (xy 87.902809 99.638583)
+						(xy 89.157118 99.638583)
 					)
 				)
 				(polygon
 					(pts
-						(xy 89.546186 99.60558) (xy 89.669506 99.645388) (xy 89.724381 99.67507) (xy 89.774884 99.711318)
-						(xy 89.822767 99.755907) (xy 89.866141 99.807633) (xy 89.907759 99.871067) (xy 89.944435 99.942787)
-						(xy 90.627582 101.446102) (xy 90.658357 101.53) (xy 90.087195 101.53) (xy 90.064976 101.466227)
-						(xy 90.064725 101.465642) (xy 89.963974 101.236053) (xy 88.843999 101.236053) (xy 88.746057 101.462833)
-						(xy 88.745853 101.463378) (xy 88.726396 101.53) (xy 88.14119 101.53) (xy 88.171965 101.446102)
-						(xy 88.454751 100.818764) (xy 89.028769 100.818764) (xy 89.779205 100.818764) (xy 89.487945 100.139281)
-						(xy 89.456926 100.097376) (xy 89.430639 100.084385) (xy 89.401239 100.080296) (xy 89.396835 100.080378)
-						(xy 89.352197 100.094063) (xy 89.333111 100.112033) (xy 89.317219 100.139281) (xy 89.028769 100.818764)
-						(xy 88.454751 100.818764) (xy 88.849616 99.942787) (xy 88.924212 99.811841) (xy 89.009949 99.717773)
-						(xy 89.058926 99.68081) (xy 89.112399 99.650285) (xy 89.172797 99.6254) (xy 89.238441 99.607374)
-						(xy 89.315148 99.595603) (xy 89.39843 99.591688)
+						(xy 91.680276 99.649453) (xy 91.761942 99.664902) (xy 91.836313 99.686626) (xy 91.905792 99.715156)
+						(xy 91.968722 99.74957) (xy 92.030486 99.793281) (xy 92.085956 99.843014) (xy 92.160789 99.931132)
+						(xy 92.235207 100.061146) (xy 92.280685 100.201712) (xy 92.295883 100.346032) (xy 92.294832 100.383887)
+						(xy 92.286587 100.458421) (xy 92.270493 100.531076) (xy 92.246338 100.602888) (xy 92.214832 100.67162)
+						(xy 92.176092 100.737193) (xy 92.130775 100.798492) (xy 92.092172 100.841013) (xy 91.983619 100.930127)
+						(xy 91.922214 100.965895) (xy 91.85486 100.996097) (xy 91.781367 101.020306) (xy 91.701373 101.038165)
+						(xy 91.613082 101.049399) (xy 91.517481 101.053237) (xy 90.646755 101.053237) (xy 90.646755 101.53)
+						(xy 90.139952 101.53) (xy 90.139952 100.178848) (xy 90.646755 100.178848) (xy 90.646755 100.588443)
+						(xy 91.528716 100.588443) (xy 91.598341 100.583348) (xy 91.644298 100.572341) (xy 91.682857 100.555599)
+						(xy 91.718389 100.530522) (xy 91.747069 100.499295) (xy 91.77719 100.446432) (xy 91.788097 100.40797)
+						(xy 91.791888 100.365572) (xy 91.782645 100.297764) (xy 91.767031 100.258598) (xy 91.744261 100.223422)
+						(xy 91.71225 100.192248) (xy 91.678858 100.170819) (xy 91.638609 100.154504) (xy 91.58839 100.143672)
+						(xy 91.528716 100.139891) (xy 90.683148 100.139891) (xy 90.661157 100.145245) (xy 90.65051 100.157832)
+						(xy 90.646755 100.178848) (xy 90.139952 100.178848) (xy 90.139952 99.756186) (xy 90.153079 99.692338)
+						(xy 90.168638 99.670423) (xy 90.190116 99.654214) (xy 90.222685 99.642491) (xy 90.263172 99.638583)
+						(xy 91.517481 99.638583)
 					)
 				)
-				(polygon
-					(pts
-						(xy 90.85888 99.638583) (xy 90.85888 101.53) (xy 91.368493 101.53) (xy 91.368493 99.638583)
-					)
-				)
-				(polygon
-					(pts
-						(xy 94.000454 99.638583) (xy 93.504885 99.638583) (xy 93.504885 100.861385) (xy 93.501221 100.88549)
-						(xy 93.491206 100.901795) (xy 93.465684 100.911699) (xy 93.440817 100.907852) (xy 93.418057 100.889351)
-						(xy 92.494086 99.779633) (xy 92.439978 99.721363) (xy 92.385079 99.67523) (xy 92.335709 99.644352)
-						(xy 92.283531 99.621201) (xy 92.167931 99.59569) (xy 92.085346 99.591688) (xy 92.008299 99.595687)
-						(xy 91.936564 99.60805) (xy 91.878454 99.626278) (xy 91.825579 99.651778) (xy 91.782604 99.681497)
-						(xy 91.744757 99.717778) (xy 91.713925 99.758554) (xy 91.688405 99.805736) (xy 91.654736 99.919745)
-						(xy 91.645709 100.034989) (xy 91.645709 101.53) (xy 92.144086 101.53) (xy 92.144086 100.245282)
-						(xy 92.147718 100.223526) (xy 92.157509 100.207092) (xy 92.190367 100.192056) (xy 92.191713 100.192037)
-						(xy 92.210418 100.195945) (xy 92.227518 100.207669) (xy 92.236532 100.217316) (xy 93.275297 101.420457)
-						(xy 93.316295 101.461968) (xy 93.361334 101.496285) (xy 93.462179 101.543754) (xy 93.585515 101.566847)
-						(xy 93.644836 101.569078) (xy 93.701864 101.56512) (xy 93.756917 101.553042) (xy 93.805675 101.534134)
-						(xy 93.850921 101.507614) (xy 93.889274 101.475722) (xy 93.923102 101.436759) (xy 93.950601 101.392636)
-						(xy 93.972686 101.341666) (xy 93.98857 101.284473) (xy 93.997982 101.220265) (xy 94.000454 101.162414)
-					)
-				)

Commit message: Fixed linking function
Used idle 40106 gate to buffer clock A before injecting it into V3205 B
Other:
- board text removed: "Up is ping-pong"
Changed lines of the file:
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@@
-		)
-	)
-	(gr_text "Up is ping-pong"
-		(at 110.514736 82.178018 0)
-		(layer "Cmts.User")
-		(effects
-			(font
-				(size 1 1)
-				(thickness 0.15)
-			)
 		)
 	)
