File: DMH_BBDelay_PCB_Main/Core_Circuit.kicad_sch (KiCad schematic)
At the start: 0 parts

Commit message: Started designing schematic
Parts:
- added R1, R28, R29: 100k, Resistor_THT:R_Axial_DIN0207_L6.3mm_D2.5mm_P7.62mm_Horizontal, symbol Device:R_US
- added R2: 1k, Resistor_THT:R_Axial_DIN0207_L6.3mm_D2.5mm_P7.62mm_Horizontal, symbol Device:R_US
- added R27: 18k, Resistor_THT:R_Axial_DIN0207_L6.3mm_D2.5mm_P7.62mm_Horizontal, symbol Device:R_US
- added R3, R4, R5: 51k, Resistor_THT:R_Axial_DIN0207_L6.3mm_D2.5mm_P7.62mm_Horizontal, symbol Device:R_US
- added R6: 47k, Resistor_THT:R_Axial_DIN0207_L6.3mm_D2.5mm_P7.62mm_Horizontal, symbol Device:R_US
- added R7: 10k, Resistor_THT:R_Axial_DIN0207_L6.3mm_D2.5mm_P7.62mm_Horizontal, symbol Device:R_US
- added R8: 82k, Resistor_THT:R_Axial_DIN0207_L6.3mm_D2.5mm_P7.62mm_Horizontal, symbol Device:R_US
- added RV14: 100k, SynthStuff:Potentiometer_Alpha_RD901F-40-00D_Single_Vertical, symbol Device:R_Potentiometer_US
- added SW1: SW_DPDT_x2, symbol Switch:SW_DPDT_x2
- added U1, U2: TL074, Package_DIP:DIP-14_W7.62mm_Socket, symbol Amplifier_Operational:TL074
- added U6: 4046, Package_DIP:DIP-16_W7.62mm_Socket, symbol 4xxx:4046
Connections:
- new net: R5.2, R6.2, R7.1, R8.1, U1.6 (-)
- new net: R7.2, U1.7
- new net: R1.2, R2.2, U1.3 (+)
- new net: R4.2, SW1.3 (C), U1.1, U1.2 (-)
- new net: R5.1, SW1.2 (B)
- new net: R28.1, RV14.2
- new net: R27.1, RV14.3
- new net: R3.2, R4.1, SW1.1 (A)
- new net +12V: R27.2
- new net -12V: R6.1
- new net Audio_In: R2.1
- new net FB_A_CV_Att: R29.1
- new net GND: R1.1, R3.1, RV14.1, U1.5 (+)
- new net VCA_FB_A/CV_Mix_In: R28.2, R29.2
- new net VCA_FB_A/Signal_Out: R8.2
Other:
- added sheet VCA_FB_A (VCA_DiffAmp_SM_Mk2_H.kicad_sch)

Commit message: Schematic in progress
Parts:
- added C12: 100nF, Capacitor_THT:C_Disc_D4.3mm_W1.9mm_P5.00mm, symbol Device:C
- added C13: 1uF Film, Capacitor_THT:C_Disc_D7.5mm_W4.4mm_P5.00mm, symbol Device:C
- added C14, C15: 220pF, Capacitor_THT:C_Disc_D3.0mm_W2.0mm_P2.50mm, symbol Device:C
- added C16: 1nF, Capacitor_THT:C_Disc_D3.0mm_W2.0mm_P2.50mm, symbol Device:C
- added D10, D6, D7, D8, D9: 1N4148, Diode_THT:D_DO-35_SOD27_P7.62mm_Horizontal, symbol Diode:1N4148
- added Q3: J113, Package_TO_SOT_SMD:SOT-23, symbol Transistor_FET:MMBFJ113
- added R30, R31: 51k, Resistor_THT:R_Axial_DIN0207_L6.3mm_D2.5mm_P7.62mm_Horizontal, symbol Device:R_US
- added R32, R33, R34, R37, R40, R43, R48, R50: 100k, Resistor_THT:R_Axial_DIN0207_L6.3mm_D2.5mm_P7.62mm_Horizontal, symbol Device:R_US
- added R35: 6k2, Resistor_THT:R_Axial_DIN0207_L6.3mm_D2.5mm_P7.62mm_Horizontal, symbol Device:R_US
- added R36, R44, R45: 10k, Resistor_THT:R_Axial_DIN0207_L6.3mm_D2.5mm_P7.62mm_Horizontal, symbol Device:R_US
- added R38: 39k, Resistor_THT:R_Axial_DIN0207_L6.3mm_D2.5mm_P7.62mm_Horizontal, symbol Device:R_US
- added R39: 2M2, Resistor_THT:R_Axial_DIN0207_L6.3mm_D2.5mm_P7.62mm_Horizontal, symbol Device:R_US
- added R46: 47k, Resistor_THT:R_Axial_DIN0207_L6.3mm_D2.5mm_P7.62mm_Horizontal, symbol Device:R_US
- added R47, R49: 33k, Resistor_THT:R_Axial_DIN0207_L6.3mm_D2.5mm_P7.62mm_Horizontal, symbol Device:R_US
- added R51: 22k, Resistor_THT:R_Axial_DIN0207_L6.3mm_D2.5mm_P7.62mm_Horizontal, symbol Device:R_US
- added RV15: B100k, SynthStuff:Potentiometer_Alpha_RD901F-40-00D_Single_Vertical, symbol Device:R_Potentiometer_US
- added SW2: SW_SPDT, symbol Switch:SW_SPDT
- added U7: V3205, Package_DIP:DIP-8-16_W7.62mm_Socket, symbol SynthStuff:V3205
- RV14: value 100k -> B100k
Connections:
- net +12V: now also R37.1, R51.2
- net -12V: now also R46.2, R49.1
- net GND: now also U2.3 (+), U2.5 (+), U6.8 (VSS), C12.1, D10.2 (A), D8.2 (A), R31.1, R32.1, R33.1, R35.1, R36.1, R38.1, R39.1, U7.1 (GND)
- net at R7.2, U1.7: now also U7.7 (In)
- net at U1.12 (+): now also C14.2, R35.2
- net at U1.13 (-): now also R36.2, R37.2
- net at U1.14: now also D6.1 (K)
- net at U2.6 (-): now also R47.2, R48.1, R50.1
- net at U2.7: now also R45.2, R47.1
- net at U2.1: now also R43.2, R44.1
- net at U2.2 (-): now also R44.2, R45.1, R46.1
- net at U6.11 (R1): now also R38.2
- net at U6.12 (R2): now also R39.2
- net +5V: now reaches U6.14 (SigIn)
- net +5V: now also U6.16 (VDD), C12.2, D7.1 (K), D9.1 (K), R30.2, U7.5 (Vdd)
- net at U6.2 (PC1): now also U7.2 (CP2)
- net at U6.3 (RefIn): now also U6.4 (FOUT), C14.1, U7.6 (CP1)
- net at U6.5 (Inh): now also D7.2 (A), D8.1 (K), R40.2
- net at U6.6 (C1): now also SW2.2 (B)
- net at U6.7 (C2): now also C15.1, C16.1
- net at U6.9 (VCOin): now also D10.1 (K), D9.2 (A), R43.1
- net at U1.10 (+): now also C13.2, R33.2
- net at U1.8: now also U1.9 (-), Q3.1 (D), R34.2
- new net: R48.2, RV15.2
- new net: R49.2, RV15.1
- new net: R51.1, RV15.3
- new net: C13.1, R32.2, U7.4 (Out2)
- new net: C16.2, SW2.1 (A)
- new net: D6.2 (A), Q3.3 (G), R34.1
- new net: R30.1, R31.2, U7.8 (Vgg)
- new net: C15.2, SW2.3 (C)
- new net Inhibt_CV: R40.1
- new net Time_A_CV_Att: R50.2
- no-connect marks 0 -> 5
Other:
- note added: "Experiment with other values to limit how long the delay time can be set with the Pot alone"
- moved on the sheet: U1C, U1D, U1E, U2A, U2B, U2C, U2D, U2E, U6

Commit message: Schematic in progress
Next is implementation of Channel B, CV Linking and Ping-Pong mode
Parts:
- added C17: 15nF, Capacitor_THT:C_Disc_D4.3mm_W1.9mm_P5.00mm, symbol Device:C
- added C18: 1uF Film, Capacitor_THT:C_Disc_D7.5mm_W4.4mm_P5.00mm, symbol Device:C
- added R41: 100k, Resistor_THT:R_Axial_DIN0207_L6.3mm_D2.5mm_P7.62mm_Horizontal, symbol Device:R_US
- added R42: 22k, Resistor_THT:R_Axial_DIN0207_L6.3mm_D2.5mm_P7.62mm_Horizontal, symbol Device:R_US
- added R84: 1k, Resistor_THT:R_Axial_DIN0207_L6.3mm_D2.5mm_P7.62mm_Horizontal, symbol Device:R_US
- added R85: 220k, Resistor_THT:R_Axial_DIN0207_L6.3mm_D2.5mm_P7.62mm_Horizontal, symbol Device:R_US
- added RV19, RV20: B100k, SynthStuff:Potentiometer_Alpha_RD901F-40-00D_Single_Vertical, symbol Device:R_Potentiometer_US
- R30: value 51k -> 4k7
- R31: value 51k -> 56k
- RV14: Function (none) -> FB A
- RV15: Function (none) -> Time A
Connections:
- net +12V: now also RV19.3
- net -12V: now also RV19.1
- net GND: now also C17.1, R42.1, RV20.1
- net VCA_FB_A/Signal_In: now also C18.2
- net VCXF_DW_A/In_A: now reaches R4.2, SW1.3 (C), U1.1, U1.2 (-)
- net at Q3.2 (S): now also U2.10 (+), C17.2
- net at U2.8: now also C18.1, R41.2
- net at U2.9 (-): now also R41.1, R42.2
- new net: R85.1, RV19.2
- new net Mix CV In: RV20.3
- new net Out: R84.2
- new net VCXF_DW_A/CV_Att_Pot: RV20.2
- new net VCXF_DW_A/CV_Mix_In: R85.2
- new net VCXF_DW_A/Out_X: R84.1
- no-connect marks 5 -> 7
Other:
- added sheet VCXF_DW_A (VC_Cross_Fader_SM_H.kicad_sch)
- title: (none) -> 3205 Delay
- moved on the sheet: U2C, U2D

Commit message: Schematic in progress
Parts:
- removed R3, R4: 51k, Resistor_THT:R_Axial_DIN0207_L6.3mm_D2.5mm_P7.62mm_Horizontal, symbol Device:R_US
- removed R51: 22k, Resistor_THT:R_Axial_DIN0207_L6.3mm_D2.5mm_P7.62mm_Horizontal, symbol Device:R_US
- added RV10: B100k, SynthStuff:Potentiometer_Alpha_RD902F-40-00D_Dual_Vertical, symbol Device:R_Potentiometer_Dual_Separate
- R46: value 47k -> 39k
- R47: value 33k -> 39k
- R48: value 100k -> 220k
- R49: value 33k -> 220k
- R5: value 51k -> 100k
- SW1: Function Gain -> Ping Pong
Connections:
- net +12V: now also RV15.3, RV10.3
- net -12V: now also RV15.1, RV10.1; no longer R49.1
- net VCXF_DW_A/In_A: now also R5.1; no longer SW1.3 (C)
- net Time_A_CV_Proc_c: now reaches R48.1, R50.1
- net Time_A_CV_Proc_c: now also R49.2; no longer R47.2, U2.6 (-)
- net at SW1.2 (B): no longer R5.1
- net Audio_In renamed A_In_m
- net FB_A_CV_Att renamed FB_A_CV_Att_c
- net Inhibt_CV renamed Inhibt_A_CV
- net Mix CV In renamed DW_A_CV_In_c
- net Out renamed DW_A_Out_m
- net Time_A_CV_Att renamed Time_A_CV_Att_c
- net VCA_FB_A/CV_Mix_In renamed FB_A_CV_Proc_c
- net VCA_FB_A/Signal_In renamed W_A_Out_m
- net VCXF_DW_A/CV_Att_Pot renamed DW_A_CV_Pot_c
- net VCXF_DW_A/CV_Mix_In renamed DW_A_Pot_c
- new net: R49.1, RV10.2
- new net Time_A_CV_Proc_m: R47.2, U2.6 (-)
Other:
- note removed: "Experiment with other values to limit how long the delay time can be set with the Pot alone"
- moved on the sheet: R27, R28, R29, R48, R5, R6, R8, R84, R85, RV14, RV15, RV19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
