File: DMH_BBDelay_PCB_Main/VC_Cross_Fader_SM_H.kicad_sch (KiCad schematic)
At the start: 47 parts, among them J3 Conn_01x04, J4 Conn_01x08, Q4 BC548, Q5 BC548, Q6 BC548, Q7 BC548, U8 TL074, U9 TL072

Commit message: Implemented Link switch in schematic
Parts:
- renumbered U9 to U12, U8 to U13
