File: DMH_BBDelay_PCB_Main/Attenuverters.kicad_sch (KiCad schematic)
At the start: 24 parts, among them U4 TL074, U5 TL072

Commit message: Schematic in progress
Other:
- company: (none) -> DMH Instruments

Commit message: Schematic in progress
Next is implementation of Channel B, CV Linking and Ping-Pong mode
Parts:
- removed C10, C11: 100nF, Capacitor_THT:C_Disc_D4.3mm_W1.9mm_P5.00mm, symbol Device:C
- removed R25, R26: 33k, Resistor_THT:R_Axial_DIN0207_L6.3mm_D2.5mm_P7.62mm_Horizontal, symbol Device:R_US
- removed RV10, RV11: 100k, SynthStuff:Potentiometer_TT_P110KH1, symbol Device:R_Potentiometer_US
- removed RV12, RV13: 50k, Potentiometer_THT:Potentiometer_Bourns_3296W_Vertical, symbol Device:R_Potentiometer_Trim_US
- removed U5: TL072, Package_DIP:DIP-8_W7.62mm_Socket, symbol Amplifier_Operational:TL072
- RV4: Function Zero Mix A CV -> Zero FB A CV
- RV5: Function Zero FB A CV -> Zero Time A CV
- RV8: Function Zero FB B CV -> Zero Time B CV
- RV9: Function Zero Mix B CV -> Zero FB B CV
Connections:
- net Mix_A_CV_Att is gone; now on net FB_A_CV_Att: RV4.2, RV4.3, U4.1
- net Mix_A_CV_In is gone; now on net FB_A_CV_In: R21.1, RV2.3
- net Mix_B_CV_Att is gone; now on net FB_B_CV_Att: RV9.2, RV9.3, U4.14
- net Mix_B_CV_In is gone; now on net FB_B_CV_In: R24.1, RV7.3
- net FB_A_CV_Att: no longer RV5.2, RV5.3, U4.7
- net FB_A_CV_In: no longer R22.1, RV3.3
- net FB_B_CV_Att: no longer RV8.2, RV8.3, U4.8
- net FB_B_CV_In: no longer R23.1, RV6.3
- net Time_A_CV_Att: now also RV5.2, RV5.3, U4.7
- net Time_A_CV_In: now also R22.1, RV3.3
- net Time_B_CV_Att: now also RV8.2, RV8.3, U4.8
- net Time_B_CV_In: now also R23.1, RV6.3
Other:
- title: (none) -> 3205 Delay

Commit message: Schematic in progress
Connections:
- net FB_A_CV_Att renamed FB_A_CV_Att_c
- net FB_A_CV_In renamed FB_A_CV_In_c
- net FB_B_CV_Att renamed FB_B_CV_Att_c
- net Time_A_CV_Att renamed Time_A_CV_Att_c
- net Time_A_CV_In renamed Time_A_CV_In_c
- net Time_B_CV_Att renamed Time_B_CV_Att_c
- net Time_B_CV_In renamed Time_B_CV_In_c
Other:
- moved on the sheet: C8, C9, R23, R24, RV6, RV7, RV8, RV9, U4C, U4D, U4E

Commit message: Implemented Link switch in schematic
Parts:
- renumbered U4 to U10

Commit message: Schematic ready for breadboarding
Connections:
- net FB_B_CV_In renamed FB_B_CV_In_c
Changed lines of the file:
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@@
 		)
 	)
-	(global_label "FB_B_CV_In"
+	(global_label "FB_B_CV_In_c"
 		(shape input)
 		(at 139.7 86.36 180)
@@
 		)
 		(property "Intersheetrefs" "${INTERSHEET_REFS}"
-			(at 126.071 86.36 0)
+			(at 124.0148 86.36 0)
 			(hide yes)
 			(show_name no)
