File: DMH_BBDelay_PCB_Main/Attenuverters.kicad_sch (KiCad schematic)
At the start: 15 parts, among them U10 TL074

Commit message: Added clock dividers for LEDs
Changed lines of the file:
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@@
 		(comment 1 "PCB for 10cm Kosmo format synthesizer module")
+	)
+	(rectangle
+		(start 19.05 25.4)
+		(end 260.35 107.95)
+		(stroke
+			(width 0.25)
+			(type dash)
+		)
+		(fill
+			(type none)
+		)
 	)
 	(junction
