File: DMH_BBDelay_PCB_Main/Compressor_B.kicad_sch (KiCad schematic)
At the start: 23 parts, among them U24 SSI2162, U25 TL074

Commit message: Designed input compressor circuits
Parts:
- removed C89, C90: 100nF, Capacitor_THT:C_Disc_D4.3mm_W1.9mm_P5.00mm, symbol Device:C
- removed D19: 1N4148, Diode_THT:D_DO-35_SOD27_P7.62mm_Horizontal, symbol Diode:1N4148
- removed U24: SSI2162, Package_SO:SSOP-10_3.9x4.9mm_P1.00mm, symbol SynthStuff:SSI2162
- added U24: SSI2162, Package_SO:SSOP-10_3.9x4.9mm_P1.00mm, symbol SynthStuff:SSI2162
- renumbered C3 to C4, C84 to C91, C85 to C92, C87 to C95, C88 to C96, C86 to C97, D21 to D23, D22 to D24, R186 to R206, R197 to R207, R198 to R208, R199 to R209, R200 to R210, R201 to R211, R202 to R212, R203 to R213, R205 to R214, R204 to R215, U25 to U26
Connections:
- net at C92.1, R208.1, U26.1: now also U24.8 (Vc_2)
- net at C97.1, R214.1, U26.13 (-): now also U24.7 (Out_2)
- net at C4.2, R207.2: now also U24.9 (In_2)
- no-connect marks 1 -> 0
