File: DMH_BBDelay_PCB_Main/VCA_DiffAmp_SM_Mk2_H.kicad_sch (KiCad schematic)
At the start: 20 parts, among them J1 Conn_01x02, J2 Conn_01x04, Q1 BC548, Q2 BC548, U3 TL072

Commit message: Schematic in progress
Other:
- company: (none) -> DMH Instruments

Commit message: Schematic in progress
Next is implementation of Channel B, CV Linking and Ping-Pong mode
Other:
- title: (none) -> 3205 Delay
Changed lines of the file:
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@@
 	(paper "A4")
 	(title_block
+		(title "3205 Delay")
 		(company "DMH Instruments")
 		(comment 1 "PCB for 10cm Kosmo format synthesizer module")

Commit message: Implemented Link switch in schematic
Parts:
- renumbered U3 to U11

Commit message: Added 10pF to Feedback VCA output stage
Parts:
- added C121: 100pF, Capacitor_THT:C_Disc_D3.0mm_W2.0mm_P2.50mm, symbol Device:C
Connections:
- net Signal_Out: now also C121.2
- net at R16.1, R20.2, U11.6 (-): now also C121.1
Other:
- note added: "Add this to the submodule!!!"
Changed lines of the file:
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@@
+	)
+	(circle
+		(center 222.25 22.86)
+		(radius 5.08)
+		(stroke
+			(width 0)
+			(type default)
+		)
+		(fill
+			(type none)
+		)
 	)
 	(circle
@@
 		)
 	)
+	(text "Add this to the submodule!!!"
+		(exclude_from_sim no)
+		(at 221.742 16.51 0)
+		(effects
+			(font
+				(size 1.27 1.27)
+			)
+		)
+	)
 	(text "Matched"
 		(exclude_from_sim no)
@@
 	)
 	(junction
+		(at 233.68 38.1)
+		(diameter 0)
+		(color 0 0 0 0)
+	)
+	(junction
 		(at 177.8 57.15)
+		(diameter 0)
+		(color 0 0 0 0)
+	)
+	(junction
+		(at 209.55 38.1)
 		(diameter 0)
 		(color 0 0 0 0)
@@
 	(wire
 		(pts
+			(xy 218.44 25.4) (xy 209.55 25.4)
+		)
+		(stroke
+			(width 0)
+			(type default)
+		)
+	)
+	(wire
+		(pts
 			(xy 190.5 88.9) (xy 190.5 91.44)
 		)
@@
 	(wire
 		(pts
+			(xy 233.68 25.4) (xy 233.68 38.1)
+		)
+		(stroke
+			(width 0)
+			(type default)
+		)
+	)
+	(wire
+		(pts
 			(xy 233.68 38.1) (xy 233.68 50.8)
 		)
@@
 	(wire
 		(pts
+			(xy 226.06 25.4) (xy 233.68 25.4)
+		)
+		(stroke
+			(width 0)
+			(type default)
+		)
+	)
+	(wire
+		(pts
 			(xy 114.3 129.54) (xy 114.3 133.35)
 		)
@@
 		(pts
 			(xy 185.42 88.9) (xy 190.5 88.9)
+		)
+		(stroke
+			(width 0)
+			(type default)
+		)
+	)
+	(wire
+		(pts
+			(xy 209.55 25.4) (xy 209.55 38.1)
 		)
 		(stroke
@@
 					(unit 1)
 				)
+			)
+		)
+	)
+	(symbol
+		(lib_id "Device:C")
+		(at 222.25 25.4 90)
+		(unit 1)
+		(body_style 1)
+		(exclude_from_sim no)
+		(in_bom yes)
+		(on_board yes)
+		(in_pos_files yes)
+		(dnp no)
+		(property "Reference" "C121"
+			(at 222.25 18.796 90)
+			(show_name no)
+			(do_not_autoplace no)
+			(effects
+				(font
+					(size 1.27 1.27)
+				)
+			)
+		)
+		(property "Value" "100pF"
+			(at 222.25 21.336 90)
+			(show_name no)
+			(do_not_autoplace no)
+			(effects
+				(font
+					(size 1.27 1.27)
+				)
+			)
+		)
+		(property "Footprint" "Capacitor_THT:C_Disc_D3.0mm_W2.0mm_P2.50mm"
+			(at 226.06 24.4348 0)
+			(hide yes)
+			(show_name no)
+			(do_not_autoplace no)
+			(effects
+				(font
+					(size 1.27 1.27)
+				)
+			)
+		)
+		(property "Datasheet" ""
+			(at 222.25 25.4 0)
+			(hide yes)
+			(show_name no)
+			(do_not_autoplace no)
+			(effects
+				(font
+					(size 1.27 1.27)
+				)
+			)
+		)
+		(property "Description" "Unpolarized capacitor"
+			(at 222.25 25.4 0)
+			(hide yes)
+			(show_name no)
+			(do_not_autoplace no)
+			(effects
+				(font
+					(size 1.27 1.27)
+				)
+			)
+		)
+		(property "Function" ""
+			(at 222.25 25.4 0)
+			(show_name no)
+			(do_not_autoplace no)
+			(effects
+				(font
+					(size 1.27 1.27)
+				)
+			)
+		)
+		(pin "1"
+		)
+		(pin "2"
+		)
+		(instances
+			(project "DMH_BBDelay_PCB_Main"
+				(path "/58f4306d-5387-4983-bb08-41a2313fd315/53120047-129a-4e0f-876f-6cafa2f18733/3af47fcf-f8fc-4281-9243-bf2820b35fa1"
+					(reference "C122")
+					(unit 1)
+				)
+				(path "/58f4306d-5387-4983-bb08-41a2313fd315/7ad2d702-dfb7-4d49-a82d-34430dd5948f/3af47fcf-f8fc-4281-9243-bf2820b35fa1"
+					(reference "C121")
+					(unit 1)
+				)

Commit message: Made feedback work
Parts:
- R10, R18: value 100k -> 10k
- R11, R15: value 100R -> 1k
- R9: value 100k -> 14k
Connections:
- net at Q2.1 (C), R14.1: now also R16.2; no longer R17.2
- net at Q1.1 (C), R12.1: now also R17.2; no longer R16.2
Other:
- note added: "This config of the VCA inverts the signal phase! Add it to the submodule"
Changed lines of the file:
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@@
 		)
 	)
+	(text "This config of the VCA inverts the signal phase!\nAdd it to the submodule"
+		(exclude_from_sim no)
+		(at 125.73 45.212 0)
+		(effects
+			(font
+				(size 1.27 1.27)
+			)
+		)
+	)
 	(text "Matched"
 		(exclude_from_sim no)
@@
 	)
 	(junction
-		(at 177.8 57.15)
+		(at 209.55 38.1)
 		(diameter 0)
 		(color 0 0 0 0)
 	)
 	(junction
-		(at 209.55 38.1)
+		(at 233.68 50.8)
 		(diameter 0)
 		(color 0 0 0 0)
 	)
 	(junction
-		(at 233.68 50.8)
+		(at 165.1 97.79)
 		(diameter 0)
 		(color 0 0 0 0)
 	)
 	(junction
-		(at 165.1 97.79)
+		(at 177.8 44.45)
 		(diameter 0)
 		(color 0 0 0 0)
@@
 	)
 	(junction
-		(at 209.55 48.26)
+		(at 152.4 57.15)
 		(diameter 0)
 		(color 0 0 0 0)
 	)
 	(junction
-		(at 209.55 53.34)
+		(at 209.55 48.26)
 		(diameter 0)
 		(color 0 0 0 0)
 	)
 	(junction
-		(at 165.1 25.4)
+		(at 209.55 53.34)
 		(diameter 0)
 		(color 0 0 0 0)
 	)
 	(junction
-		(at 152.4 44.45)
+		(at 165.1 25.4)
 		(diameter 0)
 		(color 0 0 0 0)
@@
 	(wire
 		(pts
-			(xy 177.8 57.15) (xy 177.8 83.82)
+			(xy 177.8 44.45) (xy 177.8 83.82)
 		)
 		(stroke
@@
 	(wire
 		(pts
-			(xy 177.8 57.15) (xy 193.04 57.15)
+			(xy 177.8 35.56) (xy 177.8 44.45)
 		)
 		(stroke
@@
 	(wire
 		(pts
-			(xy 152.4 44.45) (xy 152.4 83.82)
-		)
-		(stroke
-			(width 0)
-			(type default)
-		)
-	)
-	(wire
-		(pts
 			(xy 158.75 153.67) (xy 165.1 153.67)
 		)
@@
 	(wire
 		(pts
-			(xy 152.4 35.56) (xy 152.4 44.45)
+			(xy 152.4 35.56) (xy 152.4 57.15)
 		)
 		(stroke
@@
 	(wire
 		(pts
-			(xy 177.8 35.56) (xy 177.8 57.15)
-		)
-		(stroke
-			(width 0)
-			(type default)
-		)
-	)
-	(wire
-		(pts
 			(xy 209.55 53.34) (xy 209.55 59.69)
 		)
@@
 	(wire
 		(pts
-			(xy 152.4 44.45) (xy 193.04 44.45)
-		)
-		(stroke
-			(width 0)
-			(type default)
-		)
-	)
-	(wire
-		(pts
 			(xy 209.55 95.25) (xy 209.55 97.79)
 		)
@@
 	(wire
 		(pts
+			(xy 152.4 57.15) (xy 152.4 83.82)
+		)
+		(stroke
+			(width 0)
+			(type default)
+		)
+	)
+	(wire
+		(pts
 			(xy 215.9 139.7) (xy 215.9 142.24)
 		)
@@
 	(wire
 		(pts
+			(xy 152.4 57.15) (xy 193.04 57.15)
+		)
+		(stroke
+			(width 0)
+			(type default)
+		)
+	)
+	(wire
+		(pts
 			(xy 233.68 25.4) (xy 233.68 38.1)
 		)
@@
 	(wire
 		(pts
+			(xy 177.8 44.45) (xy 193.04 44.45)
+		)
+		(stroke
+			(width 0)
+			(type default)
+		)
+	)
+	(wire
+		(pts
 			(xy 209.55 105.41) (xy 209.55 107.95)
 		)
@@
 			)
 		)
-		(property "Value" "100k"
+		(property "Value" "10k"
 			(at 133.35 85.09 90)
 			(show_name no)
@@
 			)
 		)
-		(property "Value" "100k"
+		(property "Value" "14k"
 			(at 125.73 110.49 90)
 			(show_name no)
@@
 			)
 		)
-		(property "Value" "100R"
+		(property "Value" "1k"
 			(at 142.24 96.5199 0)
 			(show_name no)
@@
 			)
 		)
-		(property "Value" "100R"
+		(property "Value" "1k"
 			(at 193.04 93.9801 0)
 			(show_name no)
@@
 			)
 		)
-		(property "Value" "100k"
+		(property "Value" "10k"
 			(at 196.85 85.09 90)
 			(show_name no)

Commit message: Removed compander and adjusted feedback
Parts:
- R10, R18: value 10k -> 100k
- R11, R15: value 1k -> 100R
- R19, R20: value 100k -> 10k
- R9: value 14k -> 100k
Changed lines of the file:
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@@
 			)
 		)
-		(property "Value" "100k"
+		(property "Value" "10k"
 			(at 222.25 34.29 90)
 			(show_name no)
@@
 			)
 		)
-		(property "Value" "10k"
+		(property "Value" "100k"
 			(at 133.35 85.09 90)
 			(show_name no)
@@
 			)
 		)
-		(property "Value" "14k"
+		(property "Value" "100k"
 			(at 125.73 110.49 90)
 			(show_name no)
@@
 			)
 		)
-		(property "Value" "1k"
+		(property "Value" "100R"
 			(at 142.24 96.5199 0)
 			(show_name no)
@@
 			)
 		)
-		(property "Value" "1k"
+		(property "Value" "100R"
 			(at 193.04 93.9801 0)
 			(show_name no)
@@
 			)
 		)
-		(property "Value" "10k"
+		(property "Value" "100k"
 			(at 196.85 85.09 90)
 			(show_name no)
@@
 			)
 		)
-		(property "Value" "100k"
+		(property "Value" "10k"
 			(at 212.09 64.7699 0)
 			(show_name no)

Commit message: Synced channel A and B schematics
... and applied several minor improvements and optimizations.
Parts:
- added JP6, JP8: SolderJumper_3_Bridged12, Jumper:SolderJumper-3_P1.3mm_Bridged12_RoundedPad1.0x1.5mm_NumberLabels, symbol Jumper:SolderJumper_3_Bridged12
Connections:
- net at Q1.1 (C), R12.1: now also JP6.3 (B), JP8.1 (A); no longer R17.2
- net at Q2.1 (C), R14.1: now also JP6.1 (A), JP8.3 (B); no longer R16.2
- new net: JP8.2 (C), R17.2
- new net: JP6.2 (C), R16.2
Other:
- note added: "This config of the VCA inverts the signal phase!"
- note removed: "Add this to the submodule!!!"
- note removed: "This config of the VCA inverts the signal phase! Add it to the submodule"
- moved on the sheet: R17
