File: DMH_BBDelay_PCB_Main/Tone_Control_B.kicad_sch (KiCad schematic)
At the start: 12 parts, among them U17 TL074

Commit message: Qualified channel A on breadboard
Parts:
- R252: value 10k -> 14k
- R253: value 22k -> 56k
Changed lines of the file:
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@@
 			)
 		)
-		(property "Value" "22k"
+		(property "Value" "56k"
 			(at 139.7 104.648 90)
 			(show_name no)
@@
 			)
 		)
-		(property "Value" "10k"
+		(property "Value" "14k"
 			(at 124.46 109.2199 0)
 			(show_name no)
