File: DMH_BBDelay_PCB_Main_v2/Core_Circuit_A.kicad_sch (KiCad schematic)
At the start: 82 parts, among them J22 Conn_01x04, J23 Conn_01x04, J24 Conn_01x04, J25 Conn_01x04, J26 Conn_01x08, J27 Conn_01x08, J28 Conn_01x08, J29 Conn_01x08, Q3 J113, SW3 SW_SPDT, U1 TL074, U2 TL074, U3 V3205, U4 CD4046, U9 40106

Commit message: Preparing to design compander
Other:
- removed sheet Compressor A
