File: Simulations/Input_Filter/Output_filter_A.kicad_sch (KiCad schematic)
At the start: 14 parts, among them U21 TL072

Commit message: Fixed issue with SPICE model
Parts:
- removed U21: TL072, Package_DIP:DIP-8_W7.62mm_Socket, symbol Amplifier_Operational:TL072
- added U22: TL072, Package_DIP:DIP-8_W7.62mm_Socket, symbol Amplifier_Operational:TL072
- C69: value 33p -> 100p
- C72: value 390pF -> 220pF
- C74: value 330pF -> 1nF
Connections:
- net GND: now also U22.3 (+)
- net Out: now also U22.1
- net at C69.1, R188.2: now also U22.2 (-)
- net at R191.1: now also C116.2
- net at C72.2, R190.2: now also C73.2, R189.1
- new net +12V: U22.8 (V+)
- new net -12V: U22.4 (V-)

Commit message: Removed compander and adjusted feedback
Parts:
- R187: value 120k -> 200k
Changed lines of the file:
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@@
 			)
 		)
-		(property "Value" "120k"
+		(property "Value" "200k"
 			(at 152.4 75.692 90)
 			(show_name no)
@@
 		(unit 1)
 		(body_style 1)
-		(exclude_from_sim no)
+		(exclude_from_sim yes)
 		(in_bom yes)
 		(on_board yes)
@@
 		(unit 1)
 		(body_style 1)
-		(exclude_from_sim no)
+		(exclude_from_sim yes)
 		(in_bom yes)
 		(on_board yes)

Commit message: Synced channel A and B schematics
... and applied several minor improvements and optimizations.
Parts:
- C116: value 4.7uF -> 1uF
- C70: value 1nF -> 1.5nF
- R187: value 200k -> 120k
- R190: value 39k -> 43K
Changed lines of the file:
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@@
 			)
 		)
-		(property "Value" "1nF"
+		(property "Value" "1.5nF"
 			(at 120.65 95.25 0)
 			(show_name no)
@@
 		(unit 1)
 		(body_style 1)
-		(exclude_from_sim no)
+		(exclude_from_sim yes)
 		(in_bom yes)
 		(on_board yes)
@@
 			)
 		)
-		(property "Value" "200k"
+		(property "Value" "120k"
 			(at 152.4 75.692 90)
 			(show_name no)
@@
 			)
 		)
-		(property "Value" "39k"
+		(property "Value" "43K"
 			(at 82.55 85.852 90)
 			(show_name no)
@@
 			)
 		)
-		(property "Value" "4.7uF"
+		(property "Value" "1uF"
 			(at 57.15 83.82 90)
 			(show_name no)
