File: DMH_BBDelay_PCB_Main_v6/Compressor_A.kicad_sch (KiCad schematic)
At the start: 25 parts, among them U22 TL072, U27 SSI2162, U29 TL074

Commit message: V6 created
Parts:
- removed R230, R237: 10k, Resistor_THT:R_Axial_DIN0207_L6.3mm_D2.5mm_P7.62mm_Horizontal, symbol Device:R_US
- removed R231: 90.9k, Resistor_THT:R_Axial_DIN0207_L6.3mm_D2.5mm_P7.62mm_Horizontal, symbol Device:R_US
- removed R239, R240: 100k, Resistor_THT:R_Axial_DIN0207_L6.3mm_D2.5mm_P7.62mm_Horizontal, symbol Device:R_US
- removed RV28: 10k, Potentiometer_THT:Potentiometer_Bourns_3296X_Horizontal, symbol Device:R_Potentiometer_Trim_US
- removed U22: TL072, Package_DIP:DIP-8_W7.62mm_Socket, symbol Amplifier_Operational:TL072
- removed unit 4 of U29
- added C89, C90: 100nF, Capacitor_THT:C_Disc_D4.3mm_W1.9mm_P5.00mm, symbol Device:C
- added D19, D29, D30: 1N4148, Diode_THT:D_DO-35_SOD27_P7.62mm_Horizontal, symbol Diode:1N4148
- added R203: 90.9k, Resistor_THT:R_Axial_DIN0207_L6.3mm_D2.5mm_P7.62mm_Horizontal, symbol Device:R_US
- added R204: 10k, Resistor_THT:R_Axial_DIN0207_L6.3mm_D2.5mm_P7.62mm_Horizontal, symbol Device:R_US
- added R247: 1k, Resistor_THT:R_Axial_DIN0207_L6.3mm_D2.5mm_P7.62mm_Horizontal, symbol Device:R_US
- added unit 3 of U24
- added unit 4 of U25
- R197: renamed from R232; value 1k -> 100R
- R198: renamed from R235; value 10k -> 200k
- R205: renamed from R241; value 82k -> 62k
- renumbered C95 to C3, C96 to C84, C100 to C85, C113 to C86, C109 to C87, C111 to C88, D27 to D21, D28 to D22, R225 to R186, R238 to R199, R236 to R200, R233 to R201, R234 to R202, U27 to U24, U29 to U25
Connections:
- net +12V: now also C89.1, U24.10 (V+)
- net -12V: now also C90.1, D19.2 (A), U24.6 (V-)
- net GND: now also U25.3 (+), C89.2, C90.2, D19.1 (K), D29.1 (K), D30.2 (A), U24.5 (GND), U25.12 (+)
- net Out: now also D29.2 (A), D30.1 (K), R247.2; no longer C86.2, R205.2
- net at U25.8: now also R201.2, R202.2, R203.1; no longer C85.2
- net at R198.1, U25.1: now also C85.1, U24.3 (Vc_1); no longer U24.8 (Vc_2)
- net at R198.2, U25.2 (-): now also C85.2, R199.1, R202.1
- net at C86.1, R205.1: now also U24.4 (Out_1), U25.13 (-); no longer U24.7 (Out_2)
- net at C3.2, R197.2: now also U24.2 (In_1); no longer U24.9 (In_2)
- new net: R203.2, R204.2, U25.9 (-)
- new net: C86.2, R204.1, R205.2, R247.1, U25.14
- no-connect marks 0 -> 1
Other:
- note added: "Adding these diodes limits the compressor output to +/- 0.5V. With the added 2.5V offset at the input filter, it means V3205 input won't see excursions outside of its 2V to 3V allowed range."
- note added: "Bypassing this capacitor with a short improved the frequent loud excursions of this compressor."
- note removed: "Changed resistor from 100R to 1k, and replaced 2n2 with short"
- moved on the sheet: C85, C86, D21, D22, R199, R200, R201, R202, R205, U25B, U25C
