File: DMH_BBDelay_PCB_Main_v6/Compressor_B.kicad_sch (KiCad schematic)
At the start: 30 parts, among them U22 TL072, U24 SSI2162, U26 TL074

Commit message: V6 created
Parts:
- removed C101, C102, C104, C105: 100nF, Capacitor_THT:C_Disc_D4.3mm_W1.9mm_P5.00mm, symbol Device:C
- removed D17, D18: ZPD4v7, Diode_THT:D_DO-35_SOD27_P7.62mm_Horizontal, symbol Diode:ZPDxx
- removed R223: 90.9k, Resistor_THT:R_Axial_DIN0207_L6.3mm_D2.5mm_P7.62mm_Horizontal, symbol Device:R_US
- removed R226, R227: 10k, Resistor_THT:R_Axial_DIN0207_L6.3mm_D2.5mm_P7.62mm_Horizontal, symbol Device:R_US
- removed R228, R229: 100k, Resistor_THT:R_Axial_DIN0207_L6.3mm_D2.5mm_P7.62mm_Horizontal, symbol Device:R_US
- removed R250: 1k, Resistor_THT:R_Axial_DIN0207_L6.3mm_D2.5mm_P7.62mm_Horizontal, symbol Device:R_US
- removed RV13: 10k, Potentiometer_THT:Potentiometer_Bourns_3296X_Horizontal, symbol Device:R_Potentiometer_Trim_US
- removed U22: TL072, Package_DIP:DIP-8_W7.62mm_Socket, symbol Amplifier_Operational:TL072
- removed U24: SSI2162, Package_SO:SSOP-10_3.9x4.9mm_P1.00mm, symbol SynthStuff:SSI2162
- removed unit 4 of U26
- added C106, C107, C108, C99: 100nF, Capacitor_THT:C_Disc_D4.3mm_W1.9mm_P5.00mm, symbol Device:C
- added D20, D31, D32: 1N4148, Diode_THT:D_DO-35_SOD27_P7.62mm_Horizontal, symbol Diode:1N4148
- added R213: 90.9k, Resistor_THT:R_Axial_DIN0207_L6.3mm_D2.5mm_P7.62mm_Horizontal, symbol Device:R_US
- added R215: 10k, Resistor_THT:R_Axial_DIN0207_L6.3mm_D2.5mm_P7.62mm_Horizontal, symbol Device:R_US
- added R248: 1k, Resistor_THT:R_Axial_DIN0207_L6.3mm_D2.5mm_P7.62mm_Horizontal, symbol Device:R_US
- added U27: SSI2162, Package_SO:SSOP-10_3.9x4.9mm_P1.00mm, symbol SynthStuff:SSI2162
- added unit 4 of U28
- R207: renamed from R217; value 1k -> 100R
- R208: renamed from R218; value 10k -> 200k
- R214: renamed from R224; value 82k -> 62k
- renumbered C93 to C4, C94 to C91, C98 to C92, C103 to C97, D25 to D23, D26 to D24, R216 to R206, R219 to R209, R220 to R210, R221 to R211, R222 to R212, U26 to U28
Connections:
- net +12V: now also C107.1, C99.1, U27.10 (V+)
- net -12V: now also C106.1, C108.2, D20.2 (A), U27.6 (V-)
- net GND: now also U28.3 (+), C106.2, C107.2, C108.1, C99.2, D20.1 (K), D31.2 (A), D32.1 (K), U27.5 (GND), U28.12 (+)
- net Out: now also D31.1 (K), D32.2 (A), R248.2
- net at U28.8: now also R211.2, R212.2, R213.1; no longer C92.2
- net at R208.1, U28.1: now also C92.1, U27.3 (Vc_1)
- net at R208.2, U28.2 (-): now also C92.2, R209.1, R212.1
- net at C97.1, R214.1: now also U27.4 (Out_1), U28.13 (-)
- net at C97.2, R214.2: now also R215.1, R248.1, U28.14
- net at C4.2, R207.2: now also U27.2 (In_1)
- new net: R213.2, R215.2, U28.9 (-)
- no-connect marks 0 -> 1
Other:
- note added: "Adding these diodes limits the compressor output to +/- 0.5V. With the added 2.5V offset at the input filter, it means V3205 input won't see excursions outside of its 2V to 3V allowed range."
- note added: "Bypassing this capacitor with a short improved the frequent loud excursions of this compressor."
- note removed: "Changed resistor from 100R to 1k, and replaced 2n2 with short"
- note removed: "The attack time of this expader is way too slow for a decent plucky delay effect, but reducing the 330nF cap distorts the signal heavily. Reducing R228 from 200k to 100k helped The loos in expansion could be easily compensated with RV13."
- note removed: "Try adding zener limiting here"
- moved on the sheet: C92, C97, D23, D24, R209, R210, R211, R212, R214, U28B, U28C
