File: DMH_BBDelay_PCB_Main_v6/Expander_A.kicad_sch (KiCad schematic)
At the start: 26 parts, among them U24 SSI2162, U25 TL074

Commit message: V6 created
Parts:
- removed C89, C90: 100nF, Capacitor_THT:C_Disc_D4.3mm_W1.9mm_P5.00mm, symbol Device:C
- removed D19, D29, D30: 1N4148, Diode_THT:D_DO-35_SOD27_P7.62mm_Horizontal, symbol Diode:1N4148
- removed R203: 90.9k, Resistor_THT:R_Axial_DIN0207_L6.3mm_D2.5mm_P7.62mm_Horizontal, symbol Device:R_US
- removed R204: 10k, Resistor_THT:R_Axial_DIN0207_L6.3mm_D2.5mm_P7.62mm_Horizontal, symbol Device:R_US
- removed R247: 1k, Resistor_THT:R_Axial_DIN0207_L6.3mm_D2.5mm_P7.62mm_Horizontal, symbol Device:R_US
- removed unit 3 of U24
- removed unit 4 of U25
- added C104, C105: 100nF, Capacitor_THT:C_Disc_D4.3mm_W1.9mm_P5.00mm, symbol Device:C
- added D17, D18: ZPD4v7, Diode_THT:D_DO-35_SOD27_P7.62mm_Horizontal, symbol Diode:ZPDxx
- added R223: 90.9k, Resistor_THT:R_Axial_DIN0207_L6.3mm_D2.5mm_P7.62mm_Horizontal, symbol Device:R_US
- added R226, R227: 10k, Resistor_THT:R_Axial_DIN0207_L6.3mm_D2.5mm_P7.62mm_Horizontal, symbol Device:R_US
- added R228, R229: 100k, Resistor_THT:R_Axial_DIN0207_L6.3mm_D2.5mm_P7.62mm_Horizontal, symbol Device:R_US
- added R250: 1k, Resistor_THT:R_Axial_DIN0207_L6.3mm_D2.5mm_P7.62mm_Horizontal, symbol Device:R_US
- added RV13: 10k, Potentiometer_THT:Potentiometer_Bourns_3296X_Horizontal, symbol Device:R_Potentiometer_Trim_US
- added U22: TL072, Package_DIP:DIP-8_W7.62mm_Socket, symbol Amplifier_Operational:TL072
- added unit 4 of U26
- R217: renamed from R197; value 100R -> 1k
- R218: renamed from R198; value 200k -> 10k
- R224: renamed from R205; value 62k -> 82k
- renumbered C87 to C101, C88 to C102, C86 to C103, C3 to C93, C84 to C94, C85 to C98, D21 to D25, D22 to D26, R186 to R216, R199 to R219, R200 to R220, R201 to R221, R202 to R222, U25 to U26
Connections:
- net +12V: now also C104.1, R229.2, U22.8 (V+)
- net -12V: now also C105.2, U22.4 (V-)
- net GND: now also C104.2, C105.1, D18.2 (A), RV13.1, U22.3 (+), U26.12 (+); no longer U26.3 (+)
- net In: now also R226.1
- net Out: now also D17.2 (A), R250.2
- net at U26.9 (-): now also C98.1, R219.1, R222.2, R228.2
- net at R218.1, U26.1: now also U24.8 (Vc_2); no longer C98.1, U24.3 (Vc_1)
- net at C103.1, R224.1: now also U24.7 (Out_2), U22.2 (-); no longer U24.4 (Out_1)
- net at C103.2, R224.2: now also R250.1, U22.1
- net at C93.2, R217.2: now also U24.9 (In_2); no longer U24.2 (In_1)
- new net: C98.2, R227.2, R228.1, U26.8
- new net: R218.2, R227.1, U26.2 (-)
- new net: RV13.2, U26.3 (+)
- new net: R223.1, R226.2, U26.13 (-)
- new net: R221.2, R222.1, R223.2, U26.14
- new net: D17.1 (K), D18.1 (K)
- new net: R229.1, RV13.3
- no-connect marks 1 -> 0
Other:
- note added: "Changed resistor from 100R to 1k, and replaced 2n2 with short"
- note added: "The attack time of this expader is way too slow for a decent plucky delay effect, but reducing the 330nF cap distorts the signal heavily. Reducing R228 from 200k to 100k helped The loos in expansion could be easily compensated with RV13."
- note added: "Try adding zener limiting here"
- note removed: "Adding these diodes limits the compressor output to +/- 0.5V. With the added 2.5V offset at the input filter, it means V3205 input won't see excursions outside of its 2V to 3V allowed range."
- note removed: "Bypassing this capacitor with a short improved the frequent loud excursions of this compressor."
- moved on the sheet: C103, C98, D25, D26, R219, R220, R221, R222, R224, U26B, U26C
