File: DMH_BBDelay_PCB_Main_v6/Expander_B.kicad_sch (KiCad schematic)
At the start: 26 parts, among them U27 SSI2162, U28 TL074

Commit message: V6 created
Parts:
- removed C106, C107, C108, C99: 100nF, Capacitor_THT:C_Disc_D4.3mm_W1.9mm_P5.00mm, symbol Device:C
- removed D20, D31, D32: 1N4148, Diode_THT:D_DO-35_SOD27_P7.62mm_Horizontal, symbol Diode:1N4148
- removed R213: 90.9k, Resistor_THT:R_Axial_DIN0207_L6.3mm_D2.5mm_P7.62mm_Horizontal, symbol Device:R_US
- removed R215: 10k, Resistor_THT:R_Axial_DIN0207_L6.3mm_D2.5mm_P7.62mm_Horizontal, symbol Device:R_US
- removed R248: 1k, Resistor_THT:R_Axial_DIN0207_L6.3mm_D2.5mm_P7.62mm_Horizontal, symbol Device:R_US
- removed U27: SSI2162, Package_SO:SSOP-10_3.9x4.9mm_P1.00mm, symbol SynthStuff:SSI2162
- removed unit 4 of U28
- added C109, C111: 100nF, Capacitor_THT:C_Disc_D4.3mm_W1.9mm_P5.00mm, symbol Device:C
- added R230, R237: 10k, Resistor_THT:R_Axial_DIN0207_L6.3mm_D2.5mm_P7.62mm_Horizontal, symbol Device:R_US
- added R231: 90.9k, Resistor_THT:R_Axial_DIN0207_L6.3mm_D2.5mm_P7.62mm_Horizontal, symbol Device:R_US
- added R239, R240: 100k, Resistor_THT:R_Axial_DIN0207_L6.3mm_D2.5mm_P7.62mm_Horizontal, symbol Device:R_US
- added RV28: 10k, Potentiometer_THT:Potentiometer_Bourns_3296X_Horizontal, symbol Device:R_Potentiometer_Trim_US
- added U22: TL072, Package_DIP:DIP-8_W7.62mm_Socket, symbol Amplifier_Operational:TL072
- added U27: SSI2162, Package_SO:SSOP-10_3.9x4.9mm_P1.00mm, symbol SynthStuff:SSI2162
- added unit 4 of U29
- R232: renamed from R207; value 100R -> 1k
- R235: renamed from R208; value 200k -> 10k
- R241: renamed from R214; value 62k -> 82k
- renumbered C92 to C100, C97 to C113, C4 to C95, C91 to C96, D23 to D27, D24 to D28, R206 to R225, R211 to R233, R212 to R234, R210 to R236, R209 to R238, U28 to U29
Connections:
- net +12V: now also C109.1, R240.2
- net -12V: now also C111.2
- net GND: now also C109.2, C111.1, RV28.1, U22.5 (+), U29.12 (+); no longer U29.3 (+)
- net In: now also R230.1
- net Out: now also C113.2, R241.2, U22.7
- net at U29.9 (-): now also C100.1, R234.2, R238.1, R239.2
- net at R235.1, U29.1: now also U27.8 (Vc_2); no longer C100.1
- net at C113.1, R241.1: now also U22.6 (-), U27.7 (Out_2)
- net at C95.2, R232.2: now also U27.9 (In_2)
- new net: C100.2, R237.2, R239.1, U29.8
- new net: R235.2, R237.1, U29.2 (-)
- new net: RV28.2, U29.3 (+)
- new net: R230.2, R231.1, U29.13 (-)
- new net: R231.2, R233.2, R234.1, U29.14
- new net: R240.1, RV28.3
- no-connect marks 1 -> 0
Other:
- note added: "Changed resistor from 100R to 1k, and replaced 2n2 with short"
- note removed: "Adding these diodes limits the compressor output to +/- 0.5V. With the added 2.5V offset at the input filter, it means V3205 input won't see excursions outside of its 2V to 3V allowed range."
- note removed: "Bypassing this capacitor with a short improved the frequent loud excursions of this compressor."
- moved on the sheet: C100, C113, D27, D28, R233, R234, R236, R238, R241, U29B, U29C
